Commit message: Update Simulasi

File: catkin_ws/src/eksbot_simulation/urdf/dummy_robot.urdf.xacro (robot description, xacro)
@@ -38,9 +38,10 @@
     <origin xyz="0 0.12 -0.01" rpy="-1.5708 0 0"/>
     <axis xyz="0 0 1"/>
+    <dynamics damping="0.1" friction="0.05"/>
   </joint>
   <link name="left_wheel">
     <inertial>
-      <mass value="0.15"/>
-      <inertia ixx="0.0001" ixy="0" ixz="0" iyy="0.0001" iyz="0" izz="0.0001"/>
+      <mass value="0.2"/>
+      <inertia ixx="0.0002" ixy="0" ixz="0" iyy="0.0002" iyz="0" izz="0.0002"/>
     </inertial>
     <visual>
@@ -55,5 +56,12 @@
       </geometry>
       <surface>
-        <friction><ode><mu>1.5</mu><mu2>1.5</mu2></ode></friction>
+        <friction>
+          <ode>
+            <mu>10.0</mu>
+            <mu2>10.0</mu2>
+            <kp>1000000.0</kp>
+            <kd>10.0</kd>
+          </ode>
+        </friction>
       </surface>
     </collision>
@@ -65,9 +73,10 @@
     <origin xyz="0 -0.12 -0.01" rpy="-1.5708 0 0"/>
     <axis xyz="0 0 1"/>
+    <dynamics damping="0.1" friction="0.05"/>
   </joint>
   <link name="right_wheel">
     <inertial>
-      <mass value="0.15"/>
-      <inertia ixx="0.0001" ixy="0" ixz="0" iyy="0.0001" iyz="0" izz="0.0001"/>
+      <mass value="0.2"/>
+      <inertia ixx="0.0002" ixy="0" ixz="0" iyy="0.0002" iyz="0" izz="0.0002"/>
     </inertial>
     <visual>
@@ -82,13 +91,20 @@
       </geometry>
       <surface>
-        <friction><ode><mu>1.5</mu><mu2>1.5</mu2></ode></friction>
+        <friction>
+          <ode>
+            <mu>10.0</mu>
+            <mu2>10.0</mu2>
+            <kp>1000000.0</kp>
+            <kd>10.0</kd>
+          </ode>
+        </friction>
       </surface>
     </collision>
   </link>
-  <!-- FRONT CASTER -->
+  <!-- FRONT CASTER (Frictionless Glider - Zero Drag) -->
   <joint name="front_caster_joint" type="fixed">
     <parent link="base_link"/>
     <child link="front_caster"/>
-    <origin xyz="0.08 0 -0.03" rpy="0 0 0"/>
+    <origin xyz="0.08 0 -0.029" rpy="0 0 0"/>
   </joint>
   <link name="front_caster">
@@ -98,13 +114,22 @@
     </visual>
     <collision>
-      <geometry><sphere radius="0.02"/></geometry>
-      <surface><friction><ode><mu>0.01</mu><mu2>0.01</mu2></ode></friction></surface>
-    </collision>
-  </link>
-  <!-- REAR CASTER -->
+      <geometry><sphere radius="0.019"/></geometry>
+      <surface>
+        <friction>
+          <ode>
+            <mu>0.0</mu>
+            <mu2>0.0</mu2>
+            <slip1>1.0</slip1>
+            <slip2>1.0</slip2>
+          </ode>
+        </friction>
+      </surface>
+    </collision>
+  </link>
+  <!-- REAR CASTER (Frictionless Glider - Zero Drag) -->
   <joint name="rear_caster_joint" type="fixed">
     <parent link="base_link"/>
     <child link="rear_caster"/>
-    <origin xyz="-0.08 0 -0.03" rpy="0 0 0"/>
+    <origin xyz="-0.08 0 -0.029" rpy="0 0 0"/>
   </joint>
   <link name="rear_caster">
@@ -114,6 +139,15 @@
     </visual>
     <collision>
-      <geometry><sphere radius="0.02"/></geometry>
-      <surface><friction><ode><mu>0.01</mu><mu2>0.01</mu2></ode></friction></surface>
+      <geometry><sphere radius="0.019"/></geometry>
+      <surface>
+        <friction>
+          <ode>
+            <mu>0.0</mu>
+            <mu2>0.0</mu2>
+            <slip1>1.0</slip1>
+            <slip2>1.0</slip2>
+          </ode>
+        </friction>
+      </surface>
     </collision>
   </link>
@@ -192,5 +226,5 @@
     <parent link="mast_link"/>
     <child link="camera_link"/>
-    <origin xyz="0.01 0 0.31" rpy="0 0.25 0"/>
+    <origin xyz="0.01 0 0.31" rpy="0 0.60 0"/>
   </joint>
   <link name="camera_link">
@@ -219,6 +253,6 @@
       <wheelSeparation>0.24</wheelSeparation>
       <wheelDiameter>0.08</wheelDiameter>
-      <wheelAcceleration>1.0</wheelAcceleration>
-      <wheelTorque>10</wheelTorque>
+      <wheelAcceleration>10.0</wheelAcceleration>
+      <wheelTorque>30</wheelTorque>
       <commandTopic>cmd_vel</commandTopic>
       <odometryTopic>odom</odometryTopic>
@@ -256,3 +290,13 @@
     </sensor>
   </gazebo>
+  <!-- 3. Gazebo Vacuum Gripper Mechanism for 3D Cube Grip & Release -->
+  <gazebo>
+    <plugin name="gazebo_ros_vacuum_gripper" filename="libgazebo_ros_vacuum_gripper.so">
+      <robotNamespace>/dummy_robot</robotNamespace>
+      <bodyName>lift_carriage</bodyName>
+      <topicName>gripper_switch</topicName>
+      <maxForce>50.0</maxForce>
+      <maxDistance>0.15</maxDistance>
+    </plugin>
+  </gazebo>
 </robot>
